File: hardware/Rfid em.kicad_pcb (KiCad board)
At the start: 2 copper layers, 92.7 x 65.1 mm, 21 parts, among them IC1 EM4095, J1 Conn_01x06, U1 560uH, U2 AMS1117-5.0

Commit message: fix: Wire EM4095 per datasheet Fig. 8 and tune antenna to 134.2 kHz
Parts:
- added C11: 150 nF, Capacitor_SMD:C_0805_2012Metric, F.Cu at (111.6, 82.5)
- C2: value 1 nF -> 10 nF
- C3: value 470 nF -> 100 nF
- C4: value 100 pF -> 1 nF
- C5: value 10 nF -> 6.8 nF
- C6: value 2.5 nF -> 27 nF
- R1: value 33 kΩ -> 22 Ω; footprint Resistor_SMD:R_0805_2012Metric -> Resistor_SMD:R_2512_6332Metric
- U1: value 560uH -> ~49uH
- moved R1 19.2 mm to (125.2, 89.2), turned to 90 degrees
Connections:
- C2 pad 1: /MOD -> Net-(IC1-FCAP)
- C3 pad 1: /DEMOD_OUT -> Net-(IC1-CDEC_OUT)
- C4 pad 2: GND -> /ANT_TAP
- C6 pad 1: Net-(IC1-ANT1) -> /ANT_TAP
- IC1 pad 11: GND -> Net-(IC1-AGND)
- IC1 pad 12: GND -> /MOD
- IC1 pad 13: Net-(IC1-DMOD_OUT) -> /DEMOD_OUT
- IC1 pad 15: /MOD -> Net-(IC1-FCAP)
- IC1 pad 9: /DEMOD_OUT -> Net-(IC1-CDEC_OUT)
- R1 pad 1: Net-(IC1-DMOD_IN) -> Net-(IC1-ANT1)
- R1 pad 2: Net-(IC1-DMOD_OUT) -> Net-(U1-ANT_1)
- U1 pad 1: Net-(IC1-ANT1) -> Net-(U1-ANT_1)
- U1 pad 2: Net-(IC1-ANT2) -> /ANT_TAP
Routing:
- net /ANT_TAP: track 0.00 -> 47.1 mm, vias 0 -> 5
- net Net-(IC1-ANT2): track 52.3 -> 14.1 mm, vias 1 -> 0
- net Net-(IC1-ANT1): track 32.3 -> 7.71 mm
- net /DEMOD_OUT: track 41.3 -> 18.0 mm
- net Net-(IC1-DMOD_OUT): track 23.3 -> 0.00 mm
- net Net-(IC1-DMOD_IN): track 54.7 -> 33.1 mm
- net Net-(IC1-CDEC_OUT): track 0.00 -> 17.2 mm, vias 0 -> 2
- net GND: track 118.3 -> 109.4 mm, vias 4 -> 6
- net /MOD: track 26.0 -> 17.6 mm, vias 2 -> 1
- net Net-(IC1-FCAP): track 0.00 -> 5.03 mm, vias 0 -> 2
- net Net-(IC1-AGND): track 0.00 -> 2.28 mm
- net Net-(U1-ANT_1): track 0.00 -> 0.71 mm
Other:
- board text added: "134.2kHz RFID Reader"
- board text removed: "125kHz RFID Reader"
